Commit message: add rrt, revise urdf and rviz

File: dynamixel_arm/urdf/my_arm.urdf (robot description, URDF)
Before this commit: robot my_arm, 1 links, 0 joints
Links:
- link arm_base: geometry collision mesh filename=package://dynamixel_arm/urdf/meshes/F3.stl scale=0.001 0.001 0.001; visual mesh filename=package://dynamixel_arm/urdf/meshes/F3.stl scale=0.001 0.001 0.001

Commit message: finally work

File: dynamixel_arm/urdf/my_arm.urdf (robot description, URDF)
Before this commit: robot my_arm, 1 links, 0 joints
Links:
- added link finger_left; collision mesh filename=package://dynamixel_arm/urdf/meshes/pincher_finger.stl scale=0.01 0.01 0.01; visual mesh filename=package://dynamixel_arm/urdf/meshes/pincher_finger.stl scale=0.01 0.01 0.01
- added link finger_right; collision mesh filename=package://dynamixel_arm/urdf/meshes/pincher_finger.stl scale=0.01 0.01 0.01; visual mesh filename=package://dynamixel_arm/urdf/meshes/pincher_finger.stl scale=0.01 0.01 0.01
- added link frame_2; collision mesh filename=package://dynamixel_arm/urdf/meshes/F2.stl scale=0.001 0.001 0.001; visual mesh filename=package://dynamixel_arm/urdf/meshes/F2.stl scale=0.001 0.001 0.001
- added link frame_3_1; collision mesh filename=package://dynamixel_arm/urdf/meshes/F3.stl scale=0.001 0.001 0.001; visual mesh filename=package://dynamixel_arm/urdf/meshes/F3.stl scale=0.001 0.001 0.001
- added link frame_3_2; collision mesh filename=package://dynamixel_arm/urdf/meshes/F3.stl scale=0.001 0.001 0.001; visual mesh filename=package://dynamixel_arm/urdf/meshes/F3.stl scale=0.001 0.001 0.001
- added link frame_4; collision mesh filename=package://dynamixel_arm/urdf/meshes/F4.stl scale=0.001 0.001 0.001; visual mesh filename=package://dynamixel_arm/urdf/meshes/F4.stl scale=0.001 0.001 0.001
- added link gripper_base; collision mesh filename=package://dynamixel_arm/urdf/meshes/pincher_finger_base.stl scale=0.01 0.01 0.01; visual mesh filename=package://dynamixel_arm/urdf/meshes/pincher_finger_base.stl scale=0.01 0.01 0.01
- added link gripper_motor; collision mesh filename=package://dynamixel_arm/urdf/meshes/ax12_box.stl scale=0.001 0.001 0.001; visual mesh filename=package://dynamixel_arm/urdf/meshes/ax12_box.stl scale=0.001 0.001 0.001
- added link tilt_motor; collision mesh filename=package://dynamixel_arm/urdf/meshes/ax12_box.stl scale=0.001 0.001 0.001; visual mesh filename=package://dynamixel_arm/urdf/meshes/ax12_box.stl scale=0.001 0.001 0.001
- link arm_base: geometry collision mesh filename=package://dynamixel_arm/urdf/meshes/ax12_box.stl scale=0.001 0.001 0.001; visual mesh filename=package://dynamixel_arm/urdf/meshes/ax12_box.stl scale=0.001 0.001 0.001
Joints:
- added joint base_to_eight: type fixed, parent gripper_base, child finger_right, origin xyz=0 -0.035 0 rpy=${M_PI/2} 0 ${M_PI/2}
- added joint base_to_left: type fixed, parent gripper_base, child finger_left, origin xyz=0 0.035 0 rpy=${-M_PI/2} 0 ${-M_PI/2}
- added joint frame2toframe3_2: type fixed, parent frame_2, child frame_3_2, origin xyz=0 0 0.026 rpy=0 0 0
- added joint frame2totilt_motor: type fixed, parent tilt_motor, child frame_2, origin xyz=0 0 0.0385 rpy=0 0 0
- added joint frame4toframe3_1: type fixed, parent frame_4, child frame_3_1, origin xyz=0 0 0.052 rpy=0 0 0
- added joint gripper_joint: type fixed, parent frame_3_2, child gripper_motor, origin xyz=0 0 0.002 rpy=0 0 0
- added joint gripper_motor2base: type fixed, parent gripper_motor, child gripper_base, origin xyz=0.0175 0 0.04 rpy=0 0 0
- added joint pan_joint: type revolute, parent arm_base, child frame_4, origin xyz=0 0 0.0385 rpy=0 0 0, axis 0 0 1, limit lower=-3 upper=3 effort=1000.0 velocity=1.0
- added joint tilt_joint: type revolute, parent frame_3_1, child tilt_motor, origin xyz=0 0 0.002 rpy=0 0 0, axis 0 0 1, limit lower=-3 upper=3 effort=1000.0 velocity=1.0

Commit message: fix rotate axis and joint limit

File: dynamixel_arm/urdf/my_arm.urdf (robot description, URDF)
Before this commit: robot my_arm, 10 links, 9 joints
Joints:
- joint pan_joint: axis 0 0 1 -> 0 1 0; limit lower=-3 upper=3 effort=1000.0 velocity=1.0 -> lower=-2.9 upper=3 effort=1000.0 velocity=1.0
- joint tilt_joint: axis 0 0 1 -> 0 1 0; limit lower=-3 upper=3 effort=1000.0 velocity=1.0 -> lower=-2 upper=2 effort=1000.0 velocity=1.0

Commit message: fix joint limit

File: dynamixel_arm/urdf/my_arm.urdf (robot description, URDF)
Before this commit: robot my_arm, 10 links, 9 joints
Links:
- added link tcp
Joints:
- added joint base_to_tcp: type fixed, parent gripper_base, child tcp, origin xyz=0.04 0 0 rpy=0 0 0
- joint pan_joint: limit lower=-2.9 upper=3 effort=1000.0 velocity=1.0 -> lower=-2.617 upper=2.617 effort=1000.0 velocity=1.0
- joint tilt_joint: limit lower=-2 upper=2 effort=1000.0 velocity=1.0 -> lower=-1.78 upper=1.68 effort=1000.0 velocity=1.0

Commit message: revise fingers to prismatic joint

File: dynamixel_arm/urdf/my_arm.urdf (robot description, URDF)
Before this commit: robot my_arm, 11 links, 10 joints
Joints:
- removed joint base_to_eight
- added joint base_to_right: type prismatic, parent gripper_base, child finger_right, origin xyz=0 -0.035 0 rpy=${M_PI/2} 0 ${M_PI/2}, axis 1 0 0, limit lower=0.0 upper=0.013 effort=1000.0 velocity=1.0
- joint base_to_left: axis (none) -> 1 0 0; limit (none) -> lower=0.0 upper=0.013 effort=1000.0 velocity=1.0; type fixed -> prismatic
- joint pan_joint: limit lower=-2.617 upper=2.617 effort=1000.0 velocity=1.0 -> lower=-1.743 upper=1.948 effort=1000.0 velocity=2.0
- joint tilt_joint: limit lower=-1.78 upper=1.68 effort=1000.0 velocity=1.0 -> lower=-1.626 upper=1.79 effort=1000.0 velocity=2.0
